File: hw/MuxPi/Dyper.sch (KiCad schematic (older format))
At the start: 12 parts, among them K1 1-1462037-4, K2 1-1462037-4, P5 NS25-W2P, P6 NS25-W2P, P7 NS25-W2P, P8 NS25-W2P, Q2 2N7002, Q3 2N7002

Commit message: Add detailed info to MuxPi electronic components
The additional information includes manufacturer names and
manufacturer symbols for all components except ceramic capacitors
and resistors. It allows to create BOM (Bill Of Materials) with
actual product names.

Change-Id: Id1c518bba60322d4b8b132ad14261806070abc27
Parts:
- D2, D3: Manufacturer (none) -> TAIWAN SEMICONDUCTOR; Symbol (none) -> ES1JL
- K1, K2: Manufacturer (none) -> TE CONNECTIVITY; Symbol (none) -> 1-1462037-4
- P5, P6, P7, P8: Complementary manufacturer (none) -> NINIGI; Complementary manufacturer 1 (none) -> NINIGI; Complementary symbol (none) -> NS25-G2; Complementary symbol 1 (none) -> NS25-T; Manufacturer (none) -> NINIGI; Symbol (none) -> NS25-W2P
- Q2, Q3: Manufacturer (none) -> ON SEMICONDUCTOR (FAIRCHILD); Symbol (none) -> 2N7002

Commit message: Add alternative product for DyPer relays
Currently there is no way to buy relays originally choosen for
DyPers. Different product is added as a replacement which is widely
available at this moment.

Change-Id: If8e95ebd23554d36e86e7d23ec86ffcc953ed6df
Parts:
- K1, K2: Alt. Manufacturer (none) -> OMRON; Alt. Symbol (none) -> G6K-2F-Y 5VDC
Changed lines of the file:
@@
 EESchema Schematic File Version 4
-LIBS:MuxPi-cache
 EELAYER 26 0
 EELAYER END
@@
 F 5 "TE CONNECTIVITY" H 5750 2600 50  0001 C CNN "Manufacturer"
 F 6 "1-1462037-4" H 5750 2600 50  0001 C CNN "Symbol"
+F 7 "G6K-2F-Y 5VDC" H 5750 2600 50  0001 C CNN "Alt. Symbol"
+F 8 "OMRON" H 5750 2600 50  0001 C CNN "Alt. Manufacturer"
 	1    5750 2600
 	1    0    0    -1
@@
 F 5 "TE CONNECTIVITY" H 5750 4850 50  0001 C CNN "Manufacturer"
 F 6 "1-1462037-4" H 5750 4850 50  0001 C CNN "Symbol"
+F 7 "G6K-2F-Y 5VDC" H 5750 4850 50  0001 C CNN "Alt. Symbol"
+F 8 "OMRON" H 5750 4850 50  0001 C CNN "Alt. Manufacturer"
 	1    5750 4850
 	1    0    0    -1
