File: hw/MuxPi/Hdmi.sch (KiCad schematic (older format))
At the start: 7 parts, among them J1 471511001 (HDMI)

Commit message: Add detailed info to MuxPi electronic components
The additional information includes manufacturer names and
manufacturer symbols for all components except ceramic capacitors
and resistors. It allows to create BOM (Bill Of Materials) with
actual product names.

Change-Id: Id1c518bba60322d4b8b132ad14261806070abc27
Parts:
- J1: Manufacturer (none) -> MOLEX; Symbol (none) -> 471511001
Changed lines of the file:
@@
 F 3 "http://www.tme.eu/pl/Document/0ee89c51a17a2db3df4db584d9f4e80e/MX-47151-1001.pdf" H 5300 2600 60  0001 C CNN
 F 4 "http://www.tme.eu/pl/details/mx-47151-1001/zlacza-euro-hdmi/molex/471511001/" H 5800 3100 60  0001 C CNN "Shop link"
+F 5 "MOLEX" H 5800 3100 50  0001 C CNN "Manufacturer"
+F 6 "471511001" H 5800 3100 50  0001 C CNN "Symbol"
 	1    5800 3100
 	1    0    0    -1

Commit message: Update hardware design to version 1.3
Change-Id: I17b3f32943a6fd048f05d1b0d8676607dc54b976
Parts:
- R15: value 330R -> 10K; Shop link http://www.tme.eu/pl/details/rc0805jr-07330r/rezystory-smd-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 -> (none)
Changed lines of the file:
@@
 Sheet 4 12
 Title "MuxPi"
-Date "2018-04-20"
-Rev "1.2"
+Date "2018-08-14"
+Rev "1.3"
 Comp "SRPOL"
 Comment1 "Author: Adam Malinowski <a.malinowsk2@partner.samsung.com>"
-Comment2 "Copyright (c) 2016 - 2018 Samsung Electronics Co., Ltd All Rights Reserved"
+Comment2 "Copyright (c) 2016 -2018 Samsung Electronics Co., Ltd All Rights Reserved"
 Comment3 ""
 Comment4 ""
@@
 P 5600 4750
 F 0 "R15" H 5700 4800 50  0000 L CNN
-F 1 "330R" H 5700 4700 50  0000 L CNN
+F 1 "10K" H 5700 4700 50  0000 L CNN
 F 2 "Resistors_SMD:R_0805" V 5530 4750 50  0001 C CNN
 F 3 "http://www.tme.eu/pl/Document/7b8fed8c112f8a94930279c22c957f7f/rc0805yageo.pdf" H 5600 4750 50  0001 C CNN
-F 4 "http://www.tme.eu/pl/details/rc0805jr-07330r/rezystory-smd-0805/yageo/rc0805jr-07330rl/" V 5600 4750 60  0001 C CNN "Shop link"
 	1    5600 4750
 	1    0    0    -1
